File: NewProject_template/DevtankProject.kicad_pcb (KiCad board)
At the start: 2 copper layers, 0 parts

Commit message: Fix paths for project template libs, and setup design rules.
Other:
- net class Default: clearance 0.2 -> 0.15; via_drill 0.4 -> 0.3
- net class Fine: trace_width 0.25 -> 0.15
- net class Power added: clearance 0.2, trace_width 0.4, via_dia 0.8, via_drill 0.4
- rule trace_clearance: 0.2 -> 0.15
- rule trace_min: 0.2 -> 0.1
- rule via_min_drill: 0.2 -> 0.15
Changed lines of the file:
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@@
   (setup
     (last_trace_width 0.25)
-    (trace_clearance 0.2)
+    (user_trace_width 0.15)
+    (user_trace_width 0.25)
+    (user_trace_width 0.36)
+    (user_trace_width 0.5)
+    (user_trace_width 1)
+    (user_trace_width 2)
+    (user_trace_width 10)
+    (user_trace_width 20)
+    (trace_clearance 0.15)
     (zone_clearance 0.508)
     (zone_45_only no)
-    (trace_min 0.2)
+    (trace_min 0.1)
     (segment_width 0.2)
     (edge_width 0.15)
     (via_size 0.6)
-    (via_drill 0.4)
+    (via_drill 0.3)
     (via_min_size 0.4)
-    (via_min_drill 0.2)
+    (via_min_drill 0.15)
+    (user_via 0.4 0.2)
+    (user_via 0.6 0.3)
+    (user_via 0.8 0.4)
+    (user_via 1 0.5)
+    (user_via 1 0.75)
     (uvia_size 0.3)
     (uvia_drill 0.1)
@@
   (net 0 "")
   (net_class Default "This is the default net class."
-    (clearance 0.2)
+    (clearance 0.15)
     (trace_width 0.25)
     (via_dia 0.6)
-    (via_drill 0.4)
+    (via_drill 0.3)
     (uvia_dia 0.3)
     (uvia_drill 0.1)
@@
   (net_class Fine ""
     (clearance 0.1)
-    (trace_width 0.25)
+    (trace_width 0.15)
     (via_dia 0.4)
     (via_drill 0.2)
     (uvia_dia 0.3)
     (uvia_drill 0.1)
+  )
+  (net_class Power ""
+    (clearance 0.2)
+    (trace_width 0.4)
+    (via_dia 0.8)
+    (via_drill 0.4)
+    (uvia_dia 0.3)
+    (uvia_drill 0.1)
